File: hardware/focus-dev/control.kicad_sch (KiCad schematic)
At the start: 29 parts, among them J1 USB_C_Receptacle_USB2.0_14P, J2 Conn_01x09, J3 IDC-10, J4 Conn_01x03, SW1 SW_MEC_5G, SW2 SW_MEC_5G, U1 USBLC6-2SC6, U2 STM32H523RET6, Y1 8MHz

Commit message: wip: remove onboard encoders
Parts:
- removed SW1, SW2: SW_MEC_5G, lib:spst_6x3mm, symbol Switch:SW_MEC_5G
- added J3: IDC-14, Connector_IDC:IDC-Header_2x07_P2.54mm_Vertical, symbol Connector_Generic:Conn_02x07_Odd_Even
- added R4: 4.7k, Resistor_SMD:R_0603_1608Metric, symbol Device:R
- added R7: 1k, Resistor_SMD:R_0603_1608Metric, symbol Device:R
- added SW1, SW2: SW_Push, lib:spst_6x3mm, symbol Switch:SW_Push
- R3: value 10k -> 4.7k
- R5: value 1k -> 4.7k
- renumbered C11 to C10, C12 to C11, C10 to C12, C8 to C6, C6 to C7, C7 to C8, J3 to J1, J1 to J2, J2 to J4, J4 to J5, R4 to R6
Connections:
- net ENCODER_ANALOG is gone; now on net POWER_SENSE: U2.11 (PC3)
- net +3.3V: now also R5.1, J3.1 (Pin_1), J3.3 (Pin_3), R4.1
- net ENCODER_A: now also J3.5 (Pin_5)
- net ENCODER_B: now also J3.7 (Pin_7)
- net ENCODER_I2C_SCL: now also J3.14 (Pin_14), R4.2
- net ENCODER_I2C_SDA: now also R5.2, J3.12 (Pin_12)
- net ENCODER_INDEX: now also J3.9 (Pin_9)
- net ENCODER_SPI_CS: now also J3.10 (Pin_10)
- net ENCODER_SPI_MISO: now also J3.4 (Pin_4)
- net ENCODER_SPI_MOSI: now also J3.6 (Pin_6)
- net ENCODER_SPI_SCK: now also J3.8 (Pin_8)
- net GND: now also J3.11 (Pin_11), J3.13 (Pin_13), SW1.1, SW2.1
- net POWER_SENSE: no longer U2.24 (PC4)
- net STM_RESET: now also SW1.2
- net STM_USER_BUTTON: now also SW2.2
- net STM_USER_LED: now also R7.1; no longer R5.1
- net at D1.2 (A): now also R7.2; no longer R5.2
- net ENCODER_CTRL1: no longer names the net of U2.51 (PC10)
- net ENCODER_CTRL2: no longer names the net of U2.52 (PC11)
- net ENCODER_PWM: no longer names the net of U2.53 (PC12)
- no-connect marks 21 -> 26
Other:
- note added: "encoder interface"
- moved on the sheet: C10, C11, C12, C13, C14, C6, C7, C8, J1, J4, J5, R6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

Commit message: wip: rest of the layout
Parts:
- J4, J5: now not fitted
Connections:
- net ENCODER_SPI_MISO: now also J3.6 (Pin_6); no longer J3.4 (Pin_4)
- net ENCODER_SPI_MOSI: now also J3.4 (Pin_4); no longer J3.6 (Pin_6)
- net MOTOR_PWM_VH: now also J4.3 (Pin_3); no longer J4.4 (Pin_4)
- net MOTOR_PWM_VL: now also J4.4 (Pin_4); no longer J4.5 (Pin_5)
- net MOTOR_PWM_WH: now also J4.5 (Pin_5); no longer J4.7 (Pin_7)
- net MOTOR_PWM_WL: now also J4.6 (Pin_6); no longer J4.8 (Pin_8)
- net MOTOR_SENSE_U: now also J4.7 (Pin_7); no longer J4.3 (Pin_3)
- net MOTOR_SENSE_V: now also J4.8 (Pin_8); no longer J4.6 (Pin_6)
- net STM_USER_BUTTON: now also U2.2 (PC13); no longer U2.26 (PB0)
