File: example/hardware/focus-dev/inverter.kicad_sch (KiCad schematic)
At the start: 57 parts, among them J6 Conn_01x01, J7 Conn_01x01, J8 Conn_01x01, Q1 IPD90N04S4L04, Q2 IPD90N04S4L04, Q3 IPD90N04S4L04, Q4 IPD90N04S4L04, Q5 IPD90N04S4L04, Q6 IPD90N04S4L04, U3 INA181A3, U4 LM2105D, U5 INA181A3, U6 LM2105D, U7 INA181A3, U8 LM2105D

Commit message: decrease deadtime to 400ns
Parts:
- R10, R14, R19, R22, R28, R30: value 68 -> 33

Commit message: example: increase current measuremnt from +/-8A to +/-36A
Parts:
- C18, C23, C28: now not fitted
- R16, R24, R8: value 2m -> 1m
- R17, R25, R9: value 10 -> 0
- U3, U5, U7: value INA181A3 -> INA181A2
Changed lines of the file:
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@@
 			)
 		)
-		(property "Value" "INA181A3"
+		(property "Value" "INA181A2"
 			(at 195.834 39.37 0)
 			(show_name no)
@@
 		(on_board yes)
 		(in_pos_files yes)
-		(dnp no)
+		(dnp yes)
 		(property "Reference" "C28"
 			(at 233.68 139.6999 0)
@@
 		(on_board yes)
 		(in_pos_files yes)
-		(dnp no)
+		(dnp yes)
 		(property "Reference" "C18"
 			(at 233.68 48.2599 0)
@@
 			)
 		)
-		(property "Value" "2m"
+		(property "Value" "1m"
 			(at 177.8 90.1699 0)
 			(show_name no)
@@
 		(on_board yes)
 		(in_pos_files yes)
-		(dnp no)
+		(dnp yes)
 		(property "Reference" "C23"
 			(at 233.68 93.9799 0)
@@
 			)
 		)
-		(property "Value" "INA181A3"
+		(property "Value" "INA181A2"
 			(at 195.834 85.09 0)
 			(show_name no)
@@
 			)
 		)
-		(property "Value" "2m"
+		(property "Value" "1m"
 			(at 177.8 44.4499 0)
 			(show_name no)
@@
 			)
 		)
-		(property "Value" "10"
+		(property "Value" "0"
 			(at 223.52 86.36 90)
 			(show_name no)
@@
 			)
 		)
-		(property "Value" "10"
+		(property "Value" "0"
 			(at 223.52 132.08 90)
 			(show_name no)
@@
 			)
 		)
-		(property "Value" "INA181A3"
+		(property "Value" "INA181A2"
 			(at 195.834 130.81 0)
 			(show_name no)
@@
 			)
 		)
-		(property "Value" "10"
+		(property "Value" "0"
 			(at 223.52 40.64 90)
 			(show_name no)
@@
 			)
 		)
-		(property "Value" "2m"
+		(property "Value" "1m"
 			(at 177.8 135.8899 0)
 			(show_name no)
